File: hardware projects/bench buddy/BenchBuddy.sch (KiCad schematic (older format))
At the start: 0 parts

Commit message: TC block
Changed lines of the file:
@@
 LIBS:contrib
 LIBS:valves
+LIBS:BenchBuddy-cache
 EELAYER 27 0
 EELAYER END
@@
 Sheet 1 8
 Title ""
-Date "12 mar 2015"
+Date "13 mar 2015"
 Rev ""
 Comp ""
@@
 F1 "thermocouple.sch" 50
 F2 "TC IN +" I R 9300 2700 60
-F3 "TC IN  -" I R 9300 2850 60
-F4 "MOSI" I L 7600 2550 60
-F5 "MISO" I L 7600 2700 60
-F6 "SCLK" I L 7600 2850 60
-F7 "CS_N" I L 7600 3000 60
+F3 "MOSI" I L 7600 2550 60
+F4 "SCLK" I L 7600 2850 60
+F5 "CS_N" I L 7600 3000 60
+F6 "TC IN-" I R 9300 2850 60
+F7 "MISO" O L 7600 2700 60
 $EndSheet
 $Sheet

Commit message: FAN DRIVER
Changed lines of the file:
@@
-$EndSheet
-$Sheet
-S 7650 1050 1500 1000
-U 5500DF7B
-F0 "Fan" 50
-F1 "Fan.sch" 50
-F2 "POWER+" O R 9150 1350 60
-F3 "POWER-" I R 9150 1550 60
-F4 "TACH" I R 9150 1750 60
-F5 "TACH_OUT" O L 7650 1400 60
-F6 "FAN_IN" I L 7650 1200 60
 $EndSheet
 $Sheet
@@
 F5 "STRING-" I R 9250 4050 60
 $EndSheet
+$Sheet
+S 7650 750  1650 1250
+U 5500DF7B
+F0 "Fan" 50
+F1 "Fan.sch" 50
+F2 "POWER+" O R 9300 1050 60
+F3 "POWER-" I R 9300 1250 60
+F4 "TACH" I R 9300 1450 60
+F5 "TACH_OUT" O L 7650 1850 60
+F6 "FAN_IN" I L 7650 900 60
+F7 "CURRENT MEASURE " O L 7650 1750 60
+F8 "MOSI" I L 7650 1100 60
+F9 "MISO" O L 7650 1200 60
+F10 "CS_N" I L 7650 1300 60
+F11 "SCLK" I L 7650 1400 60
+$EndSheet
 $EndSCHEMATC

Commit message: ARDUINO DONE
Changed lines of the file:
@@
 LIBS:valves
 LIBS:BENCHBUDDEE
-LIBS:BenchBuddy-cache
+LIBS:benchbuddy-cache
 EELAYER 27 0
 EELAYER END
 $Descr A4 11693 8268
 encoding utf-8
-Sheet 1 8
+Sheet 1 9
 Title ""
-Date "14 mar 2015"
+Date "17 mar 2015"
 Rev ""
 Comp ""
@@
 $EndDescr
 $Sheet
-S 4150 3350 1500 3100
+S 7500 3300 1850 800
+U 5500DEDF
+F0 "thermocouple" 50
+F1 "thermocouple.sch" 50
+F2 "TC IN +" I R 9350 3700 60
+F3 "MOSI" I L 7500 3500 60
+F4 "SCLK" I L 7500 3800 60
+F5 "CS_N" I L 7500 3950 60
+F6 "TC IN-" I R 9350 3850 60
+F7 "MISO" O L 7500 3650 60
+$EndSheet
+$Sheet
+S 1100 1450 2200 1250
+U 5500DF28
+F0 "Power" 50
+F1 "power.sch" 50
+$EndSheet
+$Sheet
+S 9650 750  750  6150
+U 5500DFA7
+F0 "Terminal_Block" 50
+F1 "Terminal_Block.sch" 50
+F2 "V+_ADJ" I L 9650 1200 60
+F3 "V-_ADJ" I L 9650 1350 60
+F4 "FAN_OUT+" O L 9650 2150 60
+F5 "FAN_OUT-" O L 9650 2300 60
+F6 "TACH_IN" I L 9650 2450 60
+F7 "RELAY_COM" B L 9650 6400 60
+F8 "RELAY_NO" B L 9650 6250 60
+F9 "RELAY_NC" B L 9650 6100 60
+F10 "TC_IN+" O L 9650 3700 60
+F11 "TC_IN-" O L 9650 3850 60
+F12 "LED_STRING+" O L 9650 4850 60
+F13 "LED_STRING-" O L 9650 5000 60
+$EndSheet
+$Sheet
+S 7500 1950 1850 1150
+U 5500DF7B
+F0 "Fan" 50
+F1 "Fan.sch" 50
+F2 "CURRENT MEASURE " O L 7500 2950 60
+F3 "MOSI" I L 7500 2300 60
+F4 "MISO" O L 7500 2400 60
+F5 "CS_N" I L 7500 2500 60
+F6 "SCLK" I L 7500 2600 60
+F7 "TACH_IN" I R 9350 2450 60
+F8 "TACH_MEAS" O L 7500 2850 60
+F9 "FAN_EN_N" I L 7500 2100 60
+F10 "FAN_OUT-" O R 9350 2300 60
+F11 "FAN_OUT+" O R 9350 2150 60
+$EndSheet
+$Sheet
+S 5000 700  1800 1100
+U 5504E65A
+F0 "power adjustment monitor" 50
+F1 "power adjustment monitor.sch" 50
+F2 "3V3_MON" O L 5000 1200 60
+F3 "5V_MON" O L 5000 1300 60
+F4 "V+_ADJ_MONT" O L 5000 1500 60
+F5 "V-_ADJ_MON" O L 5000 1600 60
+F6 "V+_CURR_MON" O L 5000 950 60
+F7 "V-_CURR_MON" O L 5000 1050 60
+F8 "V+_ADJ" O R 6800 1200 60
+F9 "V-_ADJ" O R 6800 1350 60
+$EndSheet
+$Sheet
+S 7500 4550 1800 750
+U 5500DF53
+F0 "LED Driver" 50
+F1 "LED_Driver.sch" 50
+F2 "LED_EN_PWM" I L 7500 4650 60
+F3 "LED_STRING+" O R 9300 4850 60
+F4 "LED_STRING-" O R 9300 5000 60
+$EndSheet
+$Sheet
+S 7500 5750 1800 900
+U 5500DF06
+F0 "relay" 50
+F1 "relay.sch" 50
+F2 "RELAY_NC" B R 9300 6100 60
+F3 "RELAY_NO" B R 9300 6250 60
+F4 "RELAY_COM" B R 9300 6400 60
+F5 "RELAY+" I L 7500 6000 60
+F6 "RELAY-" O L 7500 6100 60
+$EndSheet
+Wire Wire Line
+	9650 1350 6800 1350
+Wire Wire Line
+	9650 1200 6800 1200
+Wire Wire Line
+	9650 2150 9350 2150
+Wire Wire Line
+	9650 2300 9350 2300
+Wire Wire Line
+	9650 2450 9350 2450
+Wire Wire Line
+	9650 3700 9350 3700
+Wire Wire Line
+	9650 3850 9350 3850
+Wire Wire Line
+	9650 4850 9300 4850
+Wire Wire Line
+	9650 5000 9300 5000
+Wire Wire Line
+	9650 6100 9300 6100
+Wire Wire Line
+	9650 6250 9300 6250
+Wire Wire Line
+	9650 6400 9300 6400
+Wire Wire Line
+	4600 2200 4750 2200
+Wire Wire Line
+	4750 2200 4750 950
+Wire Wire Line
+	4750 950  5000 950
+Wire Wire Line
+	4600 2350 4900 2350
+Wire Wire Line
+	4900 2350 4900 1050
+Wire Wire Line
+	4900 1050 5000 1050
+$Sheet
+S 3850 2100 750  4300
 U 5500DE97
 F0 "arduino" 50
 F1 "arduino.sch" 50
-F2 "RELAY+" O R 5650 5850 60
-F3 "RELAY-" O R 5650 5650 60
-F4 "MOSI" O R 5650 5500 60
-F5 "MISO" I R 5650 5300 60
-F6 "SCLK" O R 5650 5100 60
-F7 "CS_N" O R 5650 4850 60
-F8 "LED_EN" O R 5650 4650 60
-F9 "LED_FREQ" O R 5650 4450 60
-F10 "FAN_EN" O R 5650 3700 60
-F11 "TAC_MES" I R 5650 3950 60
-$EndSheet
-$Sheet
-S 7600 2250 1700 1000
-U 5500DEDF
-F0 "thermocouple" 50
-F1 "thermocouple.sch" 50
-F2 "TC IN +" I R 9300 2700 60
-F3 "MOSI" I L 7600 2550 60
-F4 "SCLK" I L 7600 2850 60
-F5 "CS_N" I L 7600 3000 60
-F6 "TC IN-" I R 9300 2850 60
-F7 "MISO" O L 7600 2700 60
-$EndSheet
-$Sheet
-S 7650 4950 1650 950
-U 5500DF06
-F0 "relay" 50
-F1 "relay.sch" 50
-F2 "RELAY+" I R 9300 5300 60
-F3 "RELAY-" O R 9300 5450 60
-F4 "DIN+" I L 7650 5300 60
-F5 "DIN-" O L 7650 5450 60
-$EndSheet
-$Sheet
-S 4000 1300 1600 1000
-U 5500DF28
-F0 "Power" 50
-F1 "power.sch" 50
-$EndSheet
-$Sheet
-S 9700 1350 500  5150
-U 5500DFA7
-F0 "Terminal_Block" 50
-F1 "Terminal_Block.sch" 50
-$EndSheet
-$Sheet
-S 7650 3500 1600 1100
-U 5500DF53
-F0 "LED Driver" 50
-F1 "LED_Driver.sch" 50
-F2 "EN" I L 7650 3900 60
-F3 "FREQ" I L 7650 4050 60
-F4 "STRING+" O R 9250 3900 60
-F5 "STRING-" I R 9250 4050 60
-$EndSheet
-$Sheet
-S 7650 750  1650 1250
-U 5500DF7B
-F0 "Fan" 50
-F1 "Fan.sch" 50
-F2 "POWER+" O R 9300 1050 60
-F3 "POWER-" I R 9300 1250 60
-F4 "TACH" I R 9300 1450 60
-F5 "TACH_OUT" O L 7650 1850 60
-F6 "FAN_IN" I L 7650 900 60
-F7 "CURRENT MEASURE " O L 7650 1750 60
-F8 "MOSI" I L 7650 1100 60
-F9 "MISO" O L 7650 1200 60
-F10 "CS_N" I L 7650 1300 60
-F11 "SCLK" I L 7650 1400 60
-$EndSheet
+F2 "MOSI" O R 4600 2750 60
+F3 "MISO" I R 4600 2900 60
+F4 "SCLK" O R 4600 3150 60
+F5 "RELAY+" O R 4600 6000 60
+F6 "RELAY-" O R 4600 6100 60
+F7 "FAN_EN_N" O R 4600 2600 60
+F8 "CURR_MEAS" I R 4600 3500 60
+F9 "V+_ADJ_MON" I R 4600 2200 60
+F10 "V-_ADJ_MON" I R 4600 2350 60
+F11 "LED_EN_PWN" O R 4600 4650 60
+F12 "DAC_CS_N" O R 4600 3000 60
+F13 "ADC_CS_N" O R 4600 3650 60
+F14 "TAC_MES" I R 4600 3350 60
+$EndSheet
+Wire Wire Line
+	4600 2600 5450 2600
+Wire Wire Line
+	5450 2600 5450 2100
+Wire Wire Line
+	5450 2100 7500 2100
+Wire Wire Line
+	4600 2750 5600 2750
+Wire Wire Line
+	5600 2750 5600 2300
+Wire Wire Line
+	5600 2300 7500 2300
+Wire Wire Line
+	4600 2900 5850 2900
+Wire Wire Line
+	5850 2900 5850 2400
+Wire Wire Line
+	5850 2400 7500 2400
+Wire Wire Line
+	4600 3000 6100 3000
+Wire Wire Line
+	6100 3000 6100 2500
+Wire Wire Line
+	6100 2500 7500 2500
+Wire Wire Line
+	7500 3500 7250 3500
+Wire Wire Line
+	7250 3500 7250 2300
+Connection ~ 7250 2300
+Wire Wire Line
+	7500 3650 7100 3650
+Wire Wire Line
+	7100 3650 7100 2400
+Connection ~ 7100 2400
+Wire Wire Line
+	7500 2600 6350 2600
+Wire Wire Line
+	6350 2600 6350 3150
+Wire Wire Line
+	6350 3150 4600 3150
+Connection ~ 6800 2600
+Wire Wire Line
+	7500 2850 6500 2850
+Wire Wire Line
+	6500 2850 6500 3350
+Wire Wire Line
+	6500 3350 4600 3350
+Wire Wire Line
+	7500 2950 6700 2950
+Wire Wire Line
+	6700 2950 6700 3500
+Wire Wire Line
+	6700 3500 4600 3500
+Wire Wire Line
+	6800 3800 7500 3800
+Wire Wire Line
+	6800 2600 6800 3800
+Wire Wire Line
+	7500 3950 6500 3950
+Wire Wire Line
+	6500 3950 6500 3650
+Wire Wire Line
+	6500 3650 4600 3650
+Wire Wire Line
+	4600 6000 7500 6000
+Wire Wire Line
+	7500 6100 4600 6100
+Wire Wire Line
+	7500 4650 4600 4650
 $EndSCHEMATC
