File: hardware projects/bench buddy/arduino.sch (KiCad schematic (older format))
At the start: 0 parts

Commit message: ARDUINO DONE
Parts:
- added ARD?: ARDUINOPINS, symbol ARDUINOPINS
- added R? (x13): R, ~, symbol R
Connections:
- net MISO: now also R?.2
- net MOSI: now also R?.2
- net RELAY+: now also R?.2
- net RELAY-: now also R?.2
- net SCLK: now also R?.2
- net TAC_MES: now also R?.1
- new net: ARD?.10 (ANALOGIN5), R?.2
- new net: ARD?.11 (DIGITAL0), R?.1
- new net: ARD?.12 (DIGITAL1), R?.1
- new net: ARD?.18 (DIGITAL8), R?.1
- new net: ARD?.19 (PWM0), R?.1
- new net: ARD?.20 (CS_N), R?.1
- new net: ARD?.21 (MOSI), R?.1
- new net: ARD?.22 (MISO), R?.1
- new net: ARD?.23 (SCK), R?.1
- new net: ARD?.7 (ANALOGIN2), R?.2
- new net: ARD?.8 (ANALOGIN3), R?.2
- new net: ARD?.9 (ANALOGIN4), R?.2
- new net ADC_CS_N: R?.2
- new net CURR_MEAS: R?.1
- new net DAC_CS_N: R?.2
- new net FAN_EN_N: R?.2
- new net GND: R?.1
- new net LED_EN_PWN: R?.2
- new net V+_ADJ_MON: R?.1
- new net V-_ADJ_MON: R?.1
